Commit message: now can boot two nao at once

File: gazebo_naoqi_control/models/model.xacro (robot description, xacro)
@@ -5,5 +5,5 @@
   <!-- <xacro:property name="controlPeriod" value="0.01"/> --> <!-- 100Hz control -->
   <xacro:property name="gazeboControlPeriod" value="true"/>
-  <xacro:property name="port" value="9559"/>
+  <xacro:property name="port" value="$(arg pport)"/>
   <xacro:property name="modelType" value="NAOH25V40"/>
   <!-- Include modified URDF model -->
